File: LightingBoard/CC_Buck.kicad_sch (KiCad schematic)
At the start: 21 parts, among them J2 LED Out, U2 TPS62933FDRLR, U3 INA180A2, U4 TL081HIDCKR

Commit message: almost theregit status!
Parts:
- added C17: 100nF, Capacitor_SMD:C_0603_1608Metric, symbol Device:C_Small
- renumbered C6 to C11, C7 to C12, C8 to C13, C9 to C14, C10 to C15, C11 to C16, J2 to J5, R5 to R10, R6 to R11, R7 to R12, R8 to R13, R9 to R14, R10 to R15, R12 to R16, R3 to R8, R4 to R9, U2 to U4, U3 to U5, U4 to U6
Connections:
- net +5V: now also U6.5 (V+), C17.1
- net GND: now also C17.2
- net VCC: no longer U6.5 (V+)

Commit message: woooooo finally done
Parts:
- added C11: 10u, Capacitor_SMD:C_0603_1608Metric, symbol Device:C_Small
- renumbered C11 to C10
Connections:
- net GND: now also C11.2
- net VCC: now also C11.1

Commit message: update board components
Parts:
- C10: value 10nF -> 100nF
Changed lines of the file:
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@@
 			)
 		)
-		(property "Value" "10nF"
+		(property "Value" "100nF"
 			(at 49.53 92.7162 0)
 			(effects

Commit message: less components
Parts:
- removed C16: 100nF, Capacitor_SMD:C_0603_1608Metric, symbol Device:C_Small
- removed R11, R12, R13, R14, R16: 10k, Resistor_SMD:R_0603_1608Metric, symbol Device:R_Small_US
- removed R15: 40K, Resistor_SMD:R_0603_1608Metric, symbol Device:R_Small_US
- removed U5: INA180A2, Package_TO_SOT_SMD:SOT-23-5, symbol Amplifier_Current:INA180A2
- added C41: 100nF, Capacitor_SMD:C_0603_1608Metric, symbol Device:C_Small
- added R26: 15k, Resistor_SMD:R_0603_1608Metric, symbol Device:R_Small_US
- added R27: 1k, Resistor_SMD:R_0603_1608Metric, symbol Device:R_Small_US
- U12: renamed from U6; value TL081HIDCKR -> MCP6486
- renumbered C10 to C34, C11 to C35, C12 to C36, C13 to C37, C14 to C38, C15 to C39, C17 to C40, J5 to J8, L1 to L7, L2 to L8, R8 to R23, R9 to R24, R10 to R25, U4 to U11
Connections:
- net Sum is gone; now on net FB: U12.1
- net DAC_IN: now also R26.1
- net FB: now also C41.1
- net GND: now also R27.2
- net V_sense: now also U12.3 (+)
- net at U12.4 (-): now also C41.2, R26.2, R27.1
Other:
- note added: "2.56A max current"
- moved on the sheet: C34, C35, C36, C37, C38, C39, C40, J8, L7, L8, R23, R24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

Commit message: fabbed
Parts:
- removed U12: MCP6486, Package_TO_SOT_SMD:SOT-353_SC-70-5, symbol CustomSymbols:TL081HIDCKR
- added U12: MCP6487, Package_SO:MSOP-8_3x3mm_P0.65mm, symbol Amplifier_Operational:TLV2372
- R26: value 15k -> 9k
Connections:
- net +5V: now also U12.8 (V+)
- net DAC_IN: now also C41.2, U12.2 (-); no longer R26.1
- net FB: now also U12.1
- net GND: now also U12.4 (V-)
- net V_sense: now also U12.5 (+)
- net at R26.2, R27.1: now also U12.6 (-); no longer C41.2
- new net: R26.1, U12.3 (+), U12.7
Other:
- note removed: "2.56A max current"
- moved on the sheet: C40, C41, R26, R27
