File: LightingBoard/LightingBoard.kicad_pcb (KiCad board)
At the start: 2 copper layers, 50 x 45 mm, 70 parts, among them J1 Barrel_Jack_Switch, J2 LED Out, J3 LED Out, J4 Programming, J5 UART, U1 AVR32DD20-E/REB, U10 XC6206P502MR, U2 TL5580IDR, U3 INA180A2, U4 LMR33630ADDA, U5 MCP4725xxx-xCH, U6 INA180A2, U7 LMR33630ADDA, U8 MCP4725xxx-xCH, X1 XRCGB32M000F1S2KR0

Commit message: almost theregit status!
Parts:
- removed the C10 at (145.5, 55.9)
- removed the C7 at (124.2, 56.6)
- removed the C8 at (146.6, 62.7)
- removed DAC_JPR1: SolderJumper_2_Open, Jumper:SolderJumper-2_P1.3mm_Open_RoundedPad1.0x1.5mm
- removed the J2 at (149.8, 66.5)
- removed the R3 at (146.6, 67.8)
- removed the R4 at (132.8, 67.6)
- removed the R5 at (121.4, 63.8)
- removed the R6 at (130.0, 67.6)
- removed the R7 at (135.6, 67.6)
- removed the U2 at (133.3, 73.4)
- added C25: 10nF, Capacitor_SMD:C_0603_1608Metric, F.Cu at (123.3, 74.0)
- added C26: .1u, Capacitor_SMD:C_0603_1608Metric, F.Cu at (123.3, 75.8)
- added C27: 1u, Capacitor_SMD:C_0805_2012Metric, F.Cu at (142.3, 89.5)
- added C28: 10u, Capacitor_SMD:C_0805_2012Metric, F.Cu at (140.1, 89.5)
- added C29: 100u, Capacitor_SMD:CP_Elec_6.3x7.7, F.Cu at (135.3, 87.8)
- added C30: 100nF, Capacitor_SMD:C_0603_1608Metric, F.Cu at (131.8, 80.0)
- added C31: 100nF, Capacitor_SMD:C_0603_1608Metric, F.Cu at (134.8, 74.0)
- added C32: 10nF, Capacitor_SMD:C_0603_1608Metric, F.Cu at (123.4, 52.7)
- added C33: .1u, Capacitor_SMD:C_0603_1608Metric, F.Cu at (123.4, 54.5)
- added C34: 1u, Capacitor_SMD:C_0805_2012Metric, F.Cu at (142.4, 68.2)
- added C35: 10u, Capacitor_SMD:C_0805_2012Metric, F.Cu at (140.2, 68.2)
- added C36: 100u, Capacitor_SMD:CP_Elec_6.3x7.7, F.Cu at (135.4, 66.5)
- added C37: 100nF, Capacitor_SMD:C_0603_1608Metric, F.Cu at (131.9, 58.7)
- added C38: 100nF, Capacitor_SMD:C_0603_1608Metric, F.Cu at (134.9, 52.7)
- added C4: 100nF, Capacitor_SMD:C_0603_1608Metric, F.Cu at (103.5, 90.4)
- added J5: LED Out, Connector_PinSocket_2.54mm:PinSocket_1x02_P2.54mm_Vertical, F.Cu at (141.7, 130.2)
- added J6: LED Out, Connector_PinSocket_2.54mm:PinSocket_1x02_P2.54mm_Vertical, F.Cu at (141.7, 109.1)
- added J7: LED Out, Connector_PinSocket_2.54mm:PinSocket_1x02_P2.54mm_Vertical, F.Cu at (141.6, 83.3)
- added J8: LED Out, Connector_PinSocket_2.54mm:PinSocket_1x02_P2.54mm_Vertical, F.Cu at (141.7, 62.0)
- added L5: 100uH, CustomFootprints:7447231101, F.Cu at (120.5, 86.5)
- added L6: 100uH, CustomFootprints:IND_BOURNS_SDR1307, F.Cu at (123.0, 84.5)
- added L7: 100uH, CustomFootprints:7447231101, F.Cu at (120.7, 65.2)
- added L8: 100uH, CustomFootprints:IND_BOURNS_SDR1307, F.Cu at (123.2, 63.2)
- added R1: 100k, Resistor_SMD:R_0603_1608Metric, F.Cu at (103.5, 94.6)
- added R2: 330, Resistor_SMD:R_0603_1608Metric, F.Cu at (103.4, 86.2)
- added R20: 10k, Resistor_SMD:R_0603_1608Metric, F.Cu at (134.2, 105.8)
- added R21: 10k, Resistor_SMD:R_0603_1608Metric, F.Cu at (127.2, 101.6)
- added R22: 10k, Resistor_SMD:R_0603_1608Metric, F.Cu at (139.2, 101.6)
- added R23: 10k, Resistor_SMD:R_0603_1608Metric, F.Cu at (139.2, 99.8)
- added R24: 40K, Resistor_SMD:R_0603_1608Metric, F.Cu at (130.9, 99.8)
- added R25: 10k, Resistor_SMD:R_0603_1608Metric, F.Cu at (130.9, 101.6)
- added R26: 100k, Resistor_SMD:R_0603_1608Metric, F.Cu at (127.0, 74.0)
- added R27: 100k, Resistor_SMD:R_0603_1608Metric, F.Cu at (116.5, 75.0)
- added R28: 100m, Resistor_SMD:R_1206_3216Metric, F.Cu at (142.1, 78.5)
- added R29: 10k, Resistor_SMD:R_0603_1608Metric, F.Cu at (134.1, 80.0)
- added R30: 10k, Resistor_SMD:R_0603_1608Metric, F.Cu at (127.0, 75.8)
- added R31: 10k, Resistor_SMD:R_0603_1608Metric, F.Cu at (139.1, 75.8)
- added R32: 10k, Resistor_SMD:R_0603_1608Metric, F.Cu at (139.1, 74.0)
- added R33: 40K, Resistor_SMD:R_0603_1608Metric, F.Cu at (130.8, 74.0)
- added R34: 10k, Resistor_SMD:R_0603_1608Metric, F.Cu at (130.8, 75.8)
- added R35: 100k, Resistor_SMD:R_0603_1608Metric, F.Cu at (127.2, 52.7)
- added R36: 100k, Resistor_SMD:R_0603_1608Metric, F.Cu at (116.7, 53.7)
- added R37: 100m, Resistor_SMD:R_1206_3216Metric, F.Cu at (142.2, 57.2)
- added R38: 10k, Resistor_SMD:R_0603_1608Metric, F.Cu at (134.2, 58.7)
- added R39: 10k, Resistor_SMD:R_0603_1608Metric, F.Cu at (127.2, 54.5)
- added R40: 10k, Resistor_SMD:R_0603_1608Metric, F.Cu at (139.2, 54.5)
- added R41: 10k, Resistor_SMD:R_0603_1608Metric, F.Cu at (139.2, 52.7)
- added R42: 40K, Resistor_SMD:R_0603_1608Metric, F.Cu at (130.9, 52.7)
- added R43: 10k, Resistor_SMD:R_0603_1608Metric, F.Cu at (130.9, 54.5)
- added U10: TPS62933FDRLR, Package_TO_SOT_SMD:SOT-583-8, F.Cu at (119.5, 75.0)
- added U11: INA180A2, Package_TO_SOT_SMD:SOT-23-5, F.Cu at (137.1, 80.3)
- added U12: TL081HIDCKR, Package_TO_SOT_SMD:SOT-353_SC-70-5, F.Cu at (134.8, 76.5)
- added U13: TPS62933FDRLR, Package_TO_SOT_SMD:SOT-583-8, F.Cu at (119.7, 53.7)
- added U14: INA180A2, Package_TO_SOT_SMD:SOT-23-5, F.Cu at (137.2, 59.0)
- added U15: TL081HIDCKR, Package_TO_SOT_SMD:SOT-353_SC-70-5, F.Cu at (134.9, 55.2)
- added U9: TL081HIDCKR, Package_TO_SOT_SMD:SOT-353_SC-70-5, F.Cu at (134.9, 102.3)
- C11: value 1u -> 10nF
- C12, C19: value 100nF -> .1u
- C13: value .1u -> 1u; footprint Capacitor_SMD:C_0603_1608Metric -> Capacitor_SMD:C_0805_2012Metric
- C14: value 1u -> 10u
- C15: value 10u -> 100u; footprint Capacitor_SMD:C_0805_2012Metric -> Capacitor_SMD:CP_Elec_6.3x7.7
- C16: value 100u -> 100nF; footprint Capacitor_SMD:CP_Elec_6.3x7.7 -> Capacitor_SMD:C_0603_1608Metric
- C17, C23: value 1u -> 100nF
- C18: value 100n -> 10nF
- C2: renamed from C1; value .1u -> 100n
- C20: value 10uF -> 1u; footprint Capacitor_SMD:C_0603_1608Metric -> Capacitor_SMD:C_0805_2012Metric
- C21: value 100nF -> 10u; footprint Capacitor_SMD:C_0603_1608Metric -> Capacitor_SMD:C_0805_2012Metric
- C22: value 10uF -> 100u; footprint Capacitor_SMD:C_0603_1608Metric -> Capacitor_SMD:CP_Elec_6.3x7.7
- C6: value 100nF -> 10uF
- C9: value 10u -> 100n; footprint Capacitor_SMD:C_0805_2012Metric -> Capacitor_SMD:C_0603_1608Metric
- J3: value LED Out -> UART; footprint Connector_PinSocket_2.54mm:PinSocket_1x02_P2.54mm_Vertical -> Connector_JST:JST_SH_BM04B-SRSS-TB_1x04-1MP_P1.00mm_Vertical
- J4: renamed from J5; footprint Connector_JST:JST_SH_BM04B-SRSS-TB_1x04-1MP_P1.00mm_Vertical -> Connector_PinSocket_2.54mm:PinSocket_1x04_P2.54mm_Vertical
- R10, R19: value 10k -> 100m; footprint Resistor_SMD:R_0603_1608Metric -> Resistor_SMD:R_1206_3216Metric
- R11: value 330 -> 10k
- R12: value 100m -> 10k; footprint Resistor_SMD:R_1206_3216Metric -> Resistor_SMD:R_0603_1608Metric
- R14: value 30k -> 10k
- R15: value 10k -> 40K
- R16: value 100k -> 10k
- R17, R18, R9: value 10k -> 100k
- U3: value INA180A2 -> MCP4728; footprint Package_TO_SOT_SMD:SOT-23-5 -> Package_SO:MSOP-10_3x3mm_P0.5mm
- U4, U7: value LMR33630ADDA -> TPS62933FDRLR; footprint Package_SO:Texas_HSOP-8-1EP_3.9x4.9mm_P1.27mm_ThermalVias -> Package_TO_SOT_SMD:SOT-583-8
- U5, U8: value MCP4725xxx-xCH -> INA180A2; footprint Package_TO_SOT_SMD:SOT-23-6 -> Package_TO_SOT_SMD:SOT-23-5
- U6: value INA180A2 -> TL081HIDCKR; footprint Package_TO_SOT_SMD:SOT-23-5 -> Package_TO_SOT_SMD:SOT-353_SC-70-5
- moved C2 80.7 mm to (85.4, 129.0), turned to -90 degrees
- moved L1 74.1 mm to (120.7, 133.4)
- moved L2 74.1 mm to (123.2, 131.4)
- moved J3 70.9 mm to (109.6, 23.7)
- moved U4 62.8 mm to (119.7, 122.0)
- moved J1 61.4 mm to (104.6, 126.2), turned to 90 degrees
- moved U5 61.2 mm to (137.2, 127.2), turned to 90 degrees
- moved C11 60.8 mm to (123.4, 121.0), turned to 180 degrees
- moved R9 58.2 mm to (116.7, 122.0)
- moved R10 58.0 mm to (142.2, 125.5)
- moved R8 57.3 mm to (127.2, 121.0), turned to 0 degrees
- moved R11 54.4 mm to (134.2, 127.0), turned to -90 degrees
- moved C13 53.3 mm to (142.4, 136.4), turned to -90 degrees
- moved C14 52.5 mm to (140.2, 136.4), turned to -90 degrees
- moved C15 51.0 mm to (135.4, 134.7), turned to -90 degrees
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- renumbered C25 to C1, C5 to C10, C2 to C3, C3 to C5, C4 to C7, C26 to C8, J4 to J2, R1 to R3, R2 to R4, R20 to R5, R21 to R6, R22 to R7, U10 to U2
Connections:
- C11 pad 1: GND -> /CC_Buck0/SS/PG1
- C11 pad 2: /VCC1 -> GND
- C12 pad 1: +5V -> Net-(U4-BST)
- C12 pad 2: GND -> Net-(U4-SW)
- C13 pad 1: Net-(U7-BOOT) -> /CC_Buck0/LEDOut
- C13 pad 2: Net-(U7-SW) -> GND
- C14 pad 1: /LEDOut2 -> /CC_Buck0/LEDOut
- C15 pad 1: /LEDOut2 -> /CC_Buck0/LEDOut
- C16 pad 1: /LEDOut2 -> +5V
- C17 pad 1: GND -> +5V
- C17 pad 2: /VCC2 -> GND
- C18 pad 1: GND -> /CC_Buck1/SS/PG1
- C18 pad 2: Net-(U1-PF6(*RESET)) -> GND
- C19 pad 1: +5V -> Net-(U7-BST)
- C19 pad 2: GND -> Net-(U7-SW)
- C20 pad 1: +5V -> /CC_Buck1/LEDOut
- C21 pad 1: +5V -> /CC_Buck1/LEDOut
- C22 pad 1: +5V -> /CC_Buck1/LEDOut
- C23 pad 1: VCC -> +5V
- C24 pad 1: VCC -> +5V
- C9 pad 1: /LEDOut1 -> GND
- C9 pad 2: GND -> Net-(U1-PF6(*RESET))
- J3 pad 1: /V_sense2 -> GND
- J3 pad 2: /LEDOut2 -> +5V
- L1 pad 2: /LEDOut1 -> /CC_Buck0/LEDOut
- L2 pad 2: /LEDOut1 -> /CC_Buck0/LEDOut
- L3 pad 2: /LEDOut2 -> /CC_Buck1/LEDOut
- L4 pad 2: /LEDOut2 -> /CC_Buck1/LEDOut
- R10 pad 1: GND -> /CC_Buck0/V_sense
- R10 pad 2: Net-(U2A--) -> GND
- R11 pad 1: /Reset -> Net-(U6-+)
- R11 pad 2: Net-(U1-PF6(*RESET)) -> /CC_Buck0/50*V_sense1
- R12 pad 1: /V_sense2 -> Net-(U6-+)
- R12 pad 2: GND -> /CC_Buck0/DAC_IN
- R13 pad 1: Net-(U2B-+) -> GND
- R13 pad 2: /50*V_sense2 -> Net-(U6--)
- R14 pad 1: /FB2 -> /CC_Buck0/Sum
- R14 pad 2: /Sum2 -> Net-(U6--)
- R15 pad 1: Net-(U2B-+) -> /CC_Buck0/FB
- R15 pad 2: /VDAC2 -> /CC_Buck0/Sum
- R16 pad 1: /PG2 -> GND
- R16 pad 2: /VCC2 -> /CC_Buck0/FB
- R17 pad 1: /Sum2 -> /CC_Buck1/SS/PG1
- R17 pad 2: Net-(U2B--) -> +5V
- R18 pad 2: /FB2 -> Net-(U7-RT)
- R19 pad 1: GND -> /CC_Buck1/V_sense
- R19 pad 2: Net-(U2B--) -> GND
- R3 pad 2: /SCL -> /SDA
- R4 pad 2: /SDA -> /SCL
- R8 pad 1: /PG1 -> /CC_Buck0/SS/PG1
- R8 pad 2: /VCC1 -> +5V
- R9 pad 2: /FB1 -> Net-(U4-RT)
- U1 pad 1: /Status1 -> /UART_TX0
- U1 pad 10: /UART_RX -> /Enable2
- U1 pad 11: /AVR_DAC -> /UART_TX
- U1 pad 12: unconnected-(U1-PD7-Pad12) -> /UART_RX
- U1 pad 2: /Status2 -> /UART_RX0
- U1 pad 3: /Enable1 -> unconnected-(U1-PA6-Pad3)
- U1 pad 4: /Enable2 -> unconnected-(U1-PA7-Pad4)
- U1 pad 5: /PG1 -> /Status1
- U1 pad 6: /PG2 -> /Status2
- U1 pad 7: unconnected-(U1-PC3-Pad7) -> /Enable0
- U1 pad 9: /UART_TX -> /Enable1
- U3 pad 1: /50*V_sense1 -> +5V
- U3 pad 2: GND -> /SCL
- U3 pad 3: /V_sense1 -> /SDA
- U3 pad 5: +5V -> Net-(U3-RDY/~{BSY})
- U4 pad 1: GND -> Net-(U4-RT)
- U4 pad 2: VCC -> /Enable0
- U4 pad 3: /Enable1 -> VCC
- U4 pad 4: /PG1 -> GND
- U4 pad 5: /FB1 -> Net-(U4-SW)
- U4 pad 6: /VCC1 -> Net-(U4-BST)
- U4 pad 7: Net-(U4-BOOT) -> /CC_Buck0/SS/PG1
- U4 pad 8: Net-(U4-SW) -> /CC_Buck0/FB
- U5 pad 1: /VDAC1 -> /CC_Buck0/50*V_sense1
- U5 pad 3: +5V -> /CC_Buck0/V_sense
- U5 pad 4: /SDA -> GND
- U5 pad 5: /SCL -> +5V
- U6 pad 1: /50*V_sense2 -> /CC_Buck0/Sum
- U6 pad 3: /V_sense2 -> Net-(U6-+)
- U6 pad 4: GND -> Net-(U6--)
- U7 pad 1: GND -> Net-(U7-RT)
- U7 pad 2: VCC -> /Enable1
- U7 pad 3: /Enable2 -> VCC
- U7 pad 4: /PG2 -> GND
- U7 pad 5: /FB2 -> Net-(U7-SW)
- U7 pad 6: /VCC2 -> Net-(U7-BST)
- U7 pad 7: Net-(U7-BOOT) -> /CC_Buck1/SS/PG1
- U7 pad 8: Net-(U7-SW) -> /CC_Buck1/FB
- U8 pad 1: /VDAC2 -> /CC_Buck1/50*V_sense1
- U8 pad 3: +5V -> /CC_Buck1/V_sense
- U8 pad 4: /SDA -> GND
- U8 pad 5: /SCL -> +5V
Routing:
- net +5V: track 105.7 -> 187.2 mm, vias 10 -> 14
- net GND: track 16.7 -> 88.4 mm, vias 24 -> 12
- net /Enable0: track 0.00 -> 50.9 mm, vias 0 -> 2
- net /PG2: track 33.3 -> 0.00 mm, vias 2 -> 0
- net /Sum2: track 33.0 -> 0.00 mm, vias 2 -> 0
- net /PG1: track 25.4 -> 0.00 mm, vias 2 -> 0
- net /CC_Buck2/DAC_IN: track 0.00 -> 21.8 mm, vias 0 -> 2
- net /Sum1: track 18.9 -> 0.00 mm
- net /LEDOut1: track 17.8 -> 0.00 mm
- net /AVR_DAC: track 17.5 -> 0.00 mm, vias 2 -> 0
- net /LEDOut2: track 16.4 -> 0.00 mm
- net /CC_Buck3/FB: track 0.00 -> 13.2 mm
- net /CC_Buck1/FB: track 0.00 -> 13.2 mm
- net /CC_Buck2/FB: track 0.00 -> 13.2 mm
- net /CC_Buck0/FB: track 0.00 -> 13.2 mm
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- added copper zone on F.Cu, net /CC_Buck0/LEDOut
- added copper zone on F.Cu, net /CC_Buck1/LEDOut
- added copper zone on F.Cu, net /CC_Buck2/LEDOut
- added copper zone on F.Cu, net /CC_Buck3/LEDOut
Other:
- board size 50 x 45 mm -> 45 x 90 mm
- board text added: "0"
- board text added: "1"
- board text added: "2"
- board text added: "3"

Commit message: woooooo finally done
Parts:
- removed the C3 at (97.4, 101.4)
- added C11: 10u, Capacitor_SMD:C_0603_1608Metric, F.Cu at (118.0, 122.5)
- added C19: 10u, Capacitor_SMD:C_0603_1608Metric, F.Cu at (118.0, 101.0)
- added C27: 10u, Capacitor_SMD:C_0603_1608Metric, F.Cu at (118.0, 76.5)
- added C35: 10u, Capacitor_SMD:C_0603_1608Metric, F.Cu at (118.0, 54.5)
- C2: value 100n -> 100u; footprint Capacitor_SMD:C_0805_2012Metric -> Capacitor_SMD:CP_Elec_6.3x7.7
- moved C2 78.0 mm to (111.5, 55.5), turned to 90 degrees
- moved J3 40.4 mm to (102.5, 63.5), turned to 90 degrees
- moved D2 40.1 mm to (107.5, 71.5)
- moved R7 40.0 mm to (107.5, 75.0)
- moved D1 40.0 mm to (109.5, 71.5)
- moved R6 39.9 mm to (109.5, 75.0)
- moved C3 31.9 mm to (105.0, 119.5), turned to 180 degrees
- moved J2 29.3 mm to (102.0, 104.8)
- moved J4 20.3 mm to (102.0, 79.3)
- moved C6 12.8 mm to (105.5, 98.0), turned to 90 degrees
- moved U2 12.7 mm to (108.5, 98.0)
- moved C9 12.4 mm to (111.5, 98.0)
- moved R34 2.79 mm to (133.5, 76.5)
- moved C33 2.74 mm to (137.5, 74.5)
- moved R33 2.74 mm to (133.5, 74.5)
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- renumbered C11 to C10, C19 to C20, C20 to C21, C21 to C22, C22 to C23, C23 to C24, C24 to C25, C25 to C26, C26 to C28, C27 to C29, C5 to C3, C28 to C30, C29 to C31, C30 to C32, C31 to C33, C32 to C34, C33 to C36, C34 to C37, C35 to C38, C36 to C39, C37 to C40, C38 to C41, C6 to C5, C7 to C6, C8 to C7, C9 to C8, C10 to C9
Connections:
- J2 pad 2: Net-(J2-Pin_2) -> /Reset
- J2 pad 3: /Reset -> Net-(J2-Pin_3)
- J3 pad 1: GND -> /UART_RX0
- J3 pad 2: +5V -> /UART_TX0
- J3 pad 3: /UART_TX0 -> +5V
- J3 pad 4: /UART_RX0 -> GND
- J4 pad 2: +5V -> /UART_TX
- J4 pad 3: /UART_TX -> /UART_RX
- J4 pad 4: /UART_RX -> +5V
- R5 pad 2: Net-(J2-Pin_2) -> Net-(J2-Pin_3)
- U1 pad 1: /UART_TX0 -> /Enable0
- U1 pad 10: /Enable2 -> /UART_RX0
- U1 pad 2: /UART_RX0 -> /Enable1
- U1 pad 3: unconnected-(U1-PA6-Pad3) -> /Enable2
- U1 pad 4: unconnected-(U1-PA7-Pad4) -> /Enable3
- U1 pad 7: /Enable0 -> unconnected-(U1-PC3-Pad7)
- U1 pad 9: /Enable1 -> /UART_TX0
- U13 pad 2: /Enable2 -> /Enable3
Routing:
- net /CC_Buck3/DAC_IN: track 0.00 -> 58.4 mm, vias 0 -> 4
- net /CC_Buck0/DAC_IN: track 0.00 -> 45.0 mm, vias 0 -> 4
- net /Enable3: track 0.00 -> 35.7 mm, vias 0 -> 2
- net GND: track 88.4 -> 120.4 mm, vias 12 -> 48
- net +5V: track 187.2 -> 215.3 mm, vias 14 -> 12
- net /CC_Buck1/DAC_IN: track 0.00 -> 24.7 mm, vias 0 -> 2
- net VCC: track 95.0 -> 119.1 mm, vias 6 -> 5
- net /Reset: track 0.00 -> 18.1 mm, vias 0 -> 1
- net /UART_TX0: track 0.00 -> 18.1 mm
- net /UART_RX0: track 0.00 -> 16.8 mm
- net /CC_Buck2/DAC_IN: track 21.8 -> 38.6 mm
- net Net-(J2-Pin_3): track 0.00 -> 13.3 mm, vias 0 -> 1
- net /UART_RX: track 0.00 -> 12.3 mm
- net Net-(U10-SW): track 4.45 -> 14.7 mm
- net /UPDI: track 0.00 -> 7.93 mm
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Other:
- outline, holes or cut-outs redrawn
- board text added: "5v"
- board text added: "Champers touched this board >:)"
- board text added: "RX"
- board text added: "Reset"
- board text added: "TX"
- board text added: "UPDI"

Commit message: update board components
Parts:
- C10, C18, C26, C34: value 10nF -> 100nF
- R5: value 4.7K -> 470
Changed lines of the file:
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@@
 			)
 		)
-		(property "Value" "10nF"
+		(property "Value" "100nF"
 			(at 0 1.43 0)
 			(layer "F.Fab")
@@
 			)
 		)
-		(property "Value" "4.7K"
+		(property "Value" "470"
 			(at 0 1.43 0)
 			(layer "F.Fab")
@@
 			)
 		)
-		(property "Value" "10nF"
+		(property "Value" "100nF"
 			(at 0 1.43 0)
 			(layer "F.Fab")
@@
 			)
 		)
-		(property "Value" "10nF"
+		(property "Value" "100nF"
 			(at 0 1.43 0)
 			(layer "F.Fab")
@@
 			)
 		)
-		(property "Value" "10nF"
+		(property "Value" "100nF"
 			(at 0 1.43 0)
 			(layer "F.Fab")

Commit message: less components
Parts:
- removed C4: 100nF, Capacitor_SMD:C_0603_1608Metric
- removed R28, R37: 100m, Resistor_SMD:R_1206_3216Metric
- removed R29, R30, R31, R32, R34, R38, R39, R40, R41, R43: 10k, Resistor_SMD:R_0603_1608Metric
- removed R33, R42: 40K, Resistor_SMD:R_0603_1608Metric
- removed R35, R36: 100k, Resistor_SMD:R_0603_1608Metric
- removed U13: TPS62933FDRLR, Package_TO_SOT_SMD:SOT-583-8
- removed U14: INA180A2, Package_TO_SOT_SMD:SOT-23-5
- removed U15: TL081HIDCKR, Package_TO_SOT_SMD:SOT-353_SC-70-5
- added D3: ESDA051, Diode_SMD:D_SOD-323, F.Cu at (103.0, 89.5)
- R11, R16, R21: value 10k -> 15k
- R12, R22: value 10k -> 1k
- R13, R14, R23: value 10k -> 100k
- R15: value 40K -> 100m; footprint Resistor_SMD:R_0603_1608Metric -> Resistor_SMD:R_1206_3216Metric
- R17, R27: value 100k -> 1k
- R19: value 100m -> 100k; footprint Resistor_SMD:R_1206_3216Metric -> Resistor_SMD:R_0603_1608Metric
- R20, R25: value 10k -> 100m; footprint Resistor_SMD:R_0603_1608Metric -> Resistor_SMD:R_1206_3216Metric
- R24: value 40K -> 100k
- R26: value 100k -> 15k
- U10: value TPS62933FDRLR -> MCP6486; footprint Package_TO_SOT_SMD:SOT-583-8 -> Package_TO_SOT_SMD:SOT-353_SC-70-5
- U11: value INA180A2 -> TPS62933FDRLR; footprint Package_TO_SOT_SMD:SOT-23-5 -> Package_TO_SOT_SMD:SOT-583-8
- U12, U6: value TL081HIDCKR -> MCP6486
- U5: value INA180A2 -> LM7805MPX; footprint Package_TO_SOT_SMD:SOT-23-5 -> Package_TO_SOT_SMD:SOT-223-3_TabPin2
- U8: value INA180A2 -> MCP6486; footprint Package_TO_SOT_SMD:SOT-23-5 -> Package_TO_SOT_SMD:SOT-353_SC-70-5
- U9: value TL081HIDCKR -> TPS62933FDRLR; footprint Package_TO_SOT_SMD:SOT-353_SC-70-5 -> Package_TO_SOT_SMD:SOT-583-8
- moved R24 48.7 mm to (118.2, 52.8)
- moved R25 47.5 mm to (142.0, 54.2), turned to 90 degrees
- moved R23 45.8 mm to (129.8, 54.8)
- moved U5 39.3 mm to (109.2, 100.0)
- moved R19 37.7 mm to (118.2, 75.2), turned to 0 degrees
- moved R14 32.5 mm to (118.2, 97.8)
- moved U11 31.6 mm to (122.0, 53.8), turned to 0 degrees
- moved R20 29.7 mm to (142.0, 76.8), turned to 90 degrees
- moved U9 29.6 mm to (122.0, 76.2)
- moved R21 25.8 mm to (129.8, 75.2), turned to 0 degrees
- moved R13 25.6 mm to (129.8, 99.8), turned to 0 degrees
- moved R27 25.3 mm to (133.8, 54.8)
- moved R16 25.0 mm to (129.8, 97.8), turned to 0 degrees
- moved R22 25.0 mm to (133.8, 77.2), turned to 0 degrees
- moved R18 24.7 mm to (129.8, 77.2)
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Connections:
- C16 pad 1: +5V -> /CC_Buck0/FB
- C16 pad 2: GND -> Net-(U6--)
- C25 pad 1: +5V -> /CC_Buck1/FB
- C25 pad 2: GND -> Net-(U8--)
- C28 pad 1: Net-(U10-BST) -> Net-(U9-BST)
- C28 pad 2: Net-(U10-SW) -> Net-(U9-SW)
- C33 pad 1: +5V -> /CC_Buck2/FB
- C33 pad 2: GND -> Net-(U10--)
- C36 pad 1: Net-(U13-BST) -> Net-(U11-BST)
- C36 pad 2: Net-(U13-SW) -> Net-(U11-SW)
- C41 pad 1: +5V -> /CC_Buck3/FB
- C41 pad 2: GND -> Net-(U12--)
- J1 pad 2: unconnected-(J1-Pad2) -> GND
- J1 pad 3: GND -> unconnected-(J1-Pad3)
- L5 pad 1: Net-(U10-SW) -> Net-(U9-SW)
- L6 pad 1: Net-(U10-SW) -> Net-(U9-SW)
- L7 pad 1: Net-(U13-SW) -> Net-(U11-SW)
- L8 pad 1: Net-(U13-SW) -> Net-(U11-SW)
- R11 pad 1: Net-(U6-+) -> /CC_Buck0/DAC_IN
- R11 pad 2: /CC_Buck0/50*V_sense1 -> Net-(U6--)
- R12 pad 1: Net-(U6-+) -> Net-(U6--)
- R12 pad 2: /CC_Buck0/DAC_IN -> GND
- R13 pad 1: GND -> /CC_Buck1/SS/PG1
- R13 pad 2: Net-(U6--) -> +5V
- R14 pad 1: /CC_Buck0/Sum -> GND
- R14 pad 2: Net-(U6--) -> Net-(U7-RT)
- R15 pad 1: /CC_Buck0/FB -> /CC_Buck1/V_sense
- R15 pad 2: /CC_Buck0/Sum -> GND
- R16 pad 1: GND -> /CC_Buck1/DAC_IN
- R16 pad 2: /CC_Buck0/FB -> Net-(U8--)
- R17 pad 1: /CC_Buck1/SS/PG1 -> Net-(U8--)
- R17 pad 2: +5V -> GND
- R18 pad 1: GND -> /CC_Buck2/SS/PG1
- R18 pad 2: Net-(U7-RT) -> +5V
- R19 pad 1: /CC_Buck1/V_sense -> GND
- R19 pad 2: GND -> Net-(U9-RT)
- R20 pad 1: Net-(U9-+) -> /CC_Buck2/V_sense
- R20 pad 2: /CC_Buck1/50*V_sense1 -> GND
- R21 pad 1: Net-(U9-+) -> /CC_Buck2/DAC_IN
- R21 pad 2: /CC_Buck1/DAC_IN -> Net-(U10--)
- R22 pad 1: GND -> Net-(U10--)
- R22 pad 2: Net-(U9--) -> GND
- R23 pad 1: /CC_Buck1/Sum -> /CC_Buck3/SS/PG1
- R23 pad 2: Net-(U9--) -> +5V
- R24 pad 1: /CC_Buck1/FB -> GND
- R24 pad 2: /CC_Buck1/Sum -> Net-(U11-RT)
- R25 pad 1: GND -> /CC_Buck3/V_sense
- R25 pad 2: /CC_Buck1/FB -> GND
- R26 pad 1: /CC_Buck2/SS/PG1 -> /CC_Buck3/DAC_IN
- R26 pad 2: +5V -> Net-(U12--)
- R27 pad 1: GND -> Net-(U12--)
- R27 pad 2: Net-(U10-RT) -> GND
- U10 pad 1: Net-(U10-RT) -> /CC_Buck2/FB
- U10 pad 2: /Enable2 -> GND
- U10 pad 3: VCC -> /CC_Buck2/V_sense
- U10 pad 4: GND -> Net-(U10--)
- U10 pad 5: Net-(U10-SW) -> +5V
- U11 pad 1: /CC_Buck2/50*V_sense1 -> Net-(U11-RT)
- U11 pad 2: GND -> /Enable3
- U11 pad 3: /CC_Buck2/V_sense -> VCC
- U11 pad 5: +5V -> Net-(U11-SW)
- U12 pad 1: /CC_Buck2/Sum -> /CC_Buck3/FB
- U12 pad 3: Net-(U12-+) -> /CC_Buck3/V_sense
- U5 pad 1: /CC_Buck0/50*V_sense1 -> VCC
- U5 pad 3: /CC_Buck0/V_sense -> +5V
- U6 pad 1: /CC_Buck0/Sum -> /CC_Buck0/FB
- U6 pad 3: Net-(U6-+) -> /CC_Buck0/V_sense
- U8 pad 1: /CC_Buck1/50*V_sense1 -> /CC_Buck1/FB
- U8 pad 4: GND -> Net-(U8--)
- U9 pad 1: /CC_Buck1/Sum -> Net-(U9-RT)
- U9 pad 2: GND -> /Enable2
- U9 pad 3: Net-(U9-+) -> VCC
- U9 pad 4: Net-(U9--) -> GND
- U9 pad 5: +5V -> Net-(U9-SW)
Routing:
- net GND: track 120.4 -> 76.3 mm, vias 48 -> 47
- net Net-(U9-SW): track 0.00 -> 18.9 mm
- net Net-(U11-SW): track 0.00 -> 18.9 mm
- net Net-(U10-SW): track 14.7 -> 0.00 mm
- net Net-(U13-SW): track 14.7 -> 0.00 mm
- net Net-(U8--): track 0.00 -> 10.9 mm
- net Net-(U10--): track 0.00 -> 10.9 mm
- net /CC_Buck3/Sum: track 9.50 -> 0.00 mm
- net /CC_Buck2/Sum: track 9.50 -> 0.00 mm
- net /CC_Buck1/Sum: track 9.50 -> 0.00 mm
- net /CC_Buck0/Sum: track 9.50 -> 0.00 mm
- net Net-(U15-+): track 9.07 -> 0.00 mm
- net Net-(U9-+): track 9.07 -> 0.00 mm
- net Net-(U6-+): track 9.07 -> 0.00 mm
- net Net-(U12-+): track 9.07 -> 0.00 mm
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Other:
- board text added: "5V"
- board text added: "GND"
- board text removed: "0"
- board text removed: "1"
- board text removed: "2"
- board text removed: "3"

Commit message: fabbed
Parts:
- added D4: SMBJ24A, Diode_SMD:D_SMB, F.Cu at (114.8, 128.8)
- R11, R16, R21, R26: value 15k -> 9k
- U10, U12, U6, U8: value MCP6486 -> MCP6487; footprint Package_TO_SOT_SMD:SOT-353_SC-70-5 -> Package_SO:MSOP-8_3x3mm_P0.65mm
- moved U6 5.27 mm to (136.5, 127.8)
- moved C14 4.92 mm to (142.8, 130.2), turned to -90 degrees
- moved C30 4.81 mm to (142.8, 85.2), turned to -90 degrees
- moved C38 4.81 mm to (142.8, 62.8), turned to -90 degrees
- moved C22 4.81 mm to (142.8, 107.8), turned to -90 degrees
- moved J6 4.80 mm to (142.8, 99.0)
- moved J7 4.78 mm to (142.8, 76.5)
- moved J8 4.78 mm to (142.8, 54.0)
- moved U10 4.74 mm to (136.5, 82.8)
- moved U12 4.74 mm to (136.5, 60.2)
- moved U8 4.72 mm to (136.5, 105.2)
- moved C13 4.52 mm to (140.0, 130.2), turned to -90 degrees
- moved J5 4.23 mm to (142.8, 121.5)
- moved C29 4.03 mm to (140.0, 85.2), turned to -90 degrees
- moved C37 4.03 mm to (140.0, 62.8), turned to -90 degrees
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Connections:
- C16 pad 2: Net-(U6--) -> /CC_Buck0/DAC_IN
- C25 pad 2: Net-(U8--) -> /CC_Buck1/DAC_IN
- C33 pad 2: Net-(U10--) -> /CC_Buck2/DAC_IN
- C41 pad 2: Net-(U12--) -> /CC_Buck3/DAC_IN
- R11 pad 1: /CC_Buck0/DAC_IN -> Net-(U6A-+)
- R11 pad 2: Net-(U6--) -> Net-(U6B--)
- R12 pad 1: Net-(U6--) -> Net-(U6B--)
- R16 pad 1: /CC_Buck1/DAC_IN -> Net-(U8A-+)
- R16 pad 2: Net-(U8--) -> Net-(U8B--)
- R17 pad 1: Net-(U8--) -> Net-(U8B--)
- R21 pad 1: /CC_Buck2/DAC_IN -> Net-(U10A-+)
- R21 pad 2: Net-(U10--) -> Net-(U10B--)
- R22 pad 1: Net-(U10--) -> Net-(U10B--)
- R26 pad 1: /CC_Buck3/DAC_IN -> Net-(U12A-+)
- R26 pad 2: Net-(U12--) -> Net-(U12B--)
- R27 pad 1: Net-(U12--) -> Net-(U12B--)
- U10 pad 2: GND -> /CC_Buck2/DAC_IN
- U10 pad 3: /CC_Buck2/V_sense -> Net-(U10A-+)
- U10 pad 4: Net-(U10--) -> GND
- U10 pad 5: +5V -> /CC_Buck2/V_sense
- U12 pad 2: GND -> /CC_Buck3/DAC_IN
- U12 pad 3: /CC_Buck3/V_sense -> Net-(U12A-+)
- U12 pad 4: Net-(U12--) -> GND
- U12 pad 5: +5V -> /CC_Buck3/V_sense
- U6 pad 2: GND -> /CC_Buck0/DAC_IN
- U6 pad 3: /CC_Buck0/V_sense -> Net-(U6A-+)
- U6 pad 4: Net-(U6--) -> GND
- U6 pad 5: +5V -> /CC_Buck0/V_sense
- U8 pad 2: GND -> /CC_Buck1/DAC_IN
- U8 pad 3: /CC_Buck1/V_sense -> Net-(U8A-+)
- U8 pad 4: Net-(U8--) -> GND
- U8 pad 5: +5V -> /CC_Buck1/V_sense
Routing:
- net GND: track 76.3 -> 142.0 mm, vias 47 -> 52
- net /CC_Buck0/DAC_IN: track 40.5 -> 58.4 mm
- net Net-(U6A-+): track 0.00 -> 15.8 mm
- net Net-(U12A-+): track 0.00 -> 15.8 mm
- net Net-(U8A-+): track 0.00 -> 15.8 mm
- net Net-(U10A-+): track 0.00 -> 15.8 mm
- net /CC_Buck1/DAC_IN: track 20.7 -> 36.2 mm
- net VCC: track 125.4 -> 140.4 mm
- net Net-(U8--): track 10.9 -> 0.00 mm
- net Net-(U6--): track 10.9 -> 0.00 mm
- net Net-(U12--): track 10.9 -> 0.00 mm
- net Net-(U10--): track 10.9 -> 0.00 mm
- net Net-(U8B--): track 0.00 -> 10.2 mm
- net Net-(U6B--): track 0.00 -> 10.2 mm
- net Net-(U10B--): track 0.00 -> 10.2 mm
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Other:
- board text added: "0"
- board text added: "1"
- board text added: "2"
- board text added: "3"
