File: LightingBoard/LightingBoard.kicad_sch (KiCad schematic)
At the start: 28 parts, among them J1 Barrel_Jack_Switch, J4 Programming, J5 UART, J7 UART, U10 XC6206P502MR, U14 MCP4728, U5 AVR32DD20-E/REB, X1 XRCGB32M000F1S2KR0

Commit message: almost theregit status!
Parts:
- removed TP1: TestPoint, TestPoint:TestPoint_Pad_D1.0mm, symbol Connector:TestPoint
- J4: renamed from J5; footprint Connector_JST:JST_SH_BM04B-SRSS-TB_1x04-1MP_P1.00mm_Vertical -> Connector_PinSocket_2.54mm:PinSocket_1x04_P2.54mm_Vertical
- renumbered C25 to C1, C5 to C10, C1 to C2, C2 to C3, C12 to C4, C3 to C5, C13 to C6, C4 to C7, C26 to C8, C18 to C9, J4 to J2, J7 to J3, R34 to R1, R11 to R2, R1 to R3, R2 to R4, R20 to R5, R21 to R6, R22 to R7, U5 to U1, U10 to U2, U14 to U3
Connections:
- net CC_Buck3/DAC_IN: now reaches U3.9 (VOUTD)
Other:
- added sheet CC_Buck3 (CC_Buck.kicad_sch)

Commit message: woooooo finally done
Parts:
- removed C3: 10u, Capacitor_SMD:C_0805_2012Metric, symbol Device:C_Small
- C2: value 100n -> 100u; footprint Capacitor_SMD:C_0805_2012Metric -> Capacitor_SMD:CP_Elec_6.3x7.7; Cost .01 -> .183
- renumbered C5 to C3, C6 to C5, C7 to C6, C8 to C7, C9 to C8, C10 to C9
Connections:
- net +5V: now also J3.3 (Pin_3), J4.4 (Pin_4); no longer J3.2 (Pin_2), J4.2 (Pin_2)
- net Enable0: now also U1.1 (PA4); no longer U1.7 (PC3)
- net Enable1: now also U1.2 (PA5); no longer U1.9 (PD4)
- net Enable2: now also U1.3 (PA6); no longer U1.10 (PD5)
- net GND: now also J3.4 (Pin_4); no longer J3.1 (Pin_1)
- net Reset: now also J2.2 (Pin_2); no longer J2.3 (Pin_3)
- net UART_RX: now also J4.3 (Pin_3); no longer J4.4 (Pin_4)
- net UART_RX0: now also J3.1 (Pin_1), U1.10 (PD5); no longer J3.4 (Pin_4), U1.2 (PA5)
- net UART_TX: now also J4.2 (Pin_2); no longer J4.3 (Pin_3)
- net UART_TX0: now also J3.2 (Pin_2), U1.9 (PD4); no longer J3.3 (Pin_3), U1.1 (PA4)
- net at R5.2: now also J2.3 (Pin_3); no longer J2.2 (Pin_2)
- net Enable3: now reaches U1.4 (PA7)
- no-connect marks 3 -> 2
Other:
- moved on the sheet: C3, R5

Commit message: update board components
Parts:
- R5: value 4.7K -> 470
Changed lines of the file:
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@@
 			)
 		)
-		(property "Value" "4.7K"
+		(property "Value" "470"
 			(at 121.92 185.42 90)
 			(effects

Commit message: less components
Parts:
- removed C4: 100nF, Capacitor_SMD:C_0603_1608Metric, symbol Device:C_Small
- added D3: ESDA051, Diode_SMD:D_SOD-323, symbol Diode:ESD5Zxx
- added U5: LM7805MPX, Package_TO_SOT_SMD:SOT-223-3_TabPin2, symbol Regulator_Linear:L7805
Connections:
- net +5V: now also D3.1 (K), U5.3 (OUT)
- net GND: now also J1.2, D3.2 (A), U5.2 (GND); no longer J1.3
- net VCC: now also U5.1 (IN)
Other:
- moved on the sheet: C5, C6, C9, J1, R1, U2, U3

Commit message: fabbed
Parts:
- added D4: SMBJ24A, Diode_SMD:D_SMB, symbol Diode:SMAJ24A
Connections:
- net GND: now also D4.2 (A2)
- net VCC: now also D4.1 (A1)
Changed lines of the file:
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@@
+	)
+	(junction
+		(at 66.04 52.07)
+		(diameter 0)
+		(color 0 0 0 0)
 	)
 	(junction
@@
 	(wire
 		(pts
+			(xy 59.69 52.07) (xy 66.04 52.07)
+		)
+		(stroke
+			(width 0)
+			(type default)
+		)
+	)
+	(wire
+		(pts
 			(xy 38.735 22.86) (xy 41.275 22.86)
+		)
+		(stroke
+			(width 0)
+			(type default)
+		)
+	)
+	(wire
+		(pts
+			(xy 59.69 44.45) (xy 66.04 44.45)
 		)
 		(stroke
@@
 					(unit 1)
 				)
+			)
+		)
+	)
+	(symbol
+		(lib_id "Diode:SMAJ24A")
+		(at 59.69 48.26 270)
+		(unit 1)
+		(exclude_from_sim no)
+		(in_bom yes)
+		(on_board yes)
+		(dnp no)
+		(property "Reference" "D4"
+			(at 54.864 46.99 90)
+			(effects
+				(font
+					(size 1.27 1.27)
+				)
+				(justify left)
+			)
+		)
+		(property "Value" "SMBJ24A"
+			(at 49.022 49.276 90)
+			(effects
+				(font
+					(size 1.27 1.27)
+				)
+				(justify left)
+			)
+		)
+		(property "Footprint" "Diode_SMD:D_SMB"
+			(at 54.61 48.26 0)
+			(effects
+				(font
+					(size 1.27 1.27)
+				)
+				(hide yes)
+			)
+		)
+		(property "Datasheet" "https://www.mouser.com/ProductDetail/STMicroelectronics/SMBJ24A-TR?qs=sGLxmgeNjikFvKhMTlbzxQ%3D%3D"
+			(at 59.69 46.99 0)
+			(effects
+				(font
+					(size 1.27 1.27)
+				)
+				(hide yes)
+			)
+		)
+		(property "Description" "400W unidirectional Transient Voltage Suppressor, 24.0Vr, SMA(DO-214AA)"
+			(at 59.69 48.26 0)
+			(effects
+				(font
+					(size 1.27 1.27)
+				)
+				(hide yes)
+			)
+		)
+		(pin "1"
+		)
+		(pin "2"
+		)
+		(instances
+			(project ""
+				(path "/3512c088-bc62-4a72-803d-5db96724f2eb"
+					(reference "D4")
+					(unit 1)
+				)
